File: 4ch-relay-1fan-arduino-nano-pcb.kicad_sch (KiCad schematic)
At the start: 57 parts, among them J1 Screw_Terminal_01x03, J2 Conn_01x08_Pin, J3 Screw_Terminal_01x03, J4 Screw_Terminal_01x03, J5 Screw_Terminal_01x03, J7 Conn_01x07_Pin, J9 Conn_01x04_Pin, K1 Relay_SPDT, K2 Relay_SPDT, K3 Relay_SPDT, K4 Relay_SPDT, Q1 2N3904, Q2 2N3904, Q3 2N3904, Q4 2N3904, Q5 BT136, U1 PC817, U2 PC817, U3 PC817, U4 PC817, U5 MOC3021M, U6 PC817, U7 TSOP1738

Commit message: Add files via upload
Parts:
- added U8: HLK-10M05, Converter_ACDC:Converter_ACDC_Hi-Link_HLK-10Mxx, symbol Converter_ACDC:HLK-10M05
Connections:
- net +5V: now also U8.4 (+Vout)
- net GND: now also U8.3 (-Vout)
- net at BR1.4, J6.2 (Pin_2), J8.1 (Pin_1): now also U8.2 (AC/N)
- net at C1.2, J6.1 (Pin_1), Q5.1 (A1)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: now also U8.1 (AC/L)
Other:
- moved on the sheet: BR1, C1, D1, D2, D3, D4, D5, D6, D7, D8, J1, J2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
