File: 4ch-relay-1fan-arduino-nano-pcb.kicad_pcb (KiCad board)
At the start: 2 copper layers, 57 parts, among them J1 Screw_Terminal_01x03, J2 Conn_01x08_Pin, J3 Screw_Terminal_01x03, J4 Screw_Terminal_01x03, J5 Screw_Terminal_01x03, J7 Conn_01x07_Pin, J9 Conn_01x04_Pin, K1 Relay_SPDT, K2 Relay_SPDT, K3 Relay_SPDT, K4 Relay_SPDT, Q1 2N3904, Q2 2N3904, Q3 2N3904, Q4 2N3904, Q5 BT136, U1 PC817, U2 PC817, U3 PC817, U4 PC817, U5 MOC3021M, U6 PC817, U7 TSOP1738

Commit message: Add files via upload
Parts:
- added U8: HLK-10M05, Converter_ACDC:Converter_ACDC_Hi-Link_HLK-10Mxx, F.Cu at (195.1, 101.6)
- moved J7 2.26 mm to (151.1, 141.3)
- moved D1 2.26 mm to (167.5, 93.3)
- moved R4 2.26 mm to (152.9, 97.0)
- moved R5 2.26 mm to (130.2, 97.0)
- moved U1 2.26 mm to (157.7, 91.6)
- moved U2 2.26 mm to (135.0, 91.6)
- moved U5 2.26 mm to (177.0, 86.1)
- moved A1 2.26 mm to (116.2, 132.2)
- moved J9 2.26 mm to (111.2, 141.2)
- moved R10 2.26 mm to (118.0, 83.7)
- moved R14 2.26 mm to (94.5, 83.4)
- moved D5 2.26 mm to (122.0, 93.3)
- moved D6 2.26 mm to (120.3, 74.5)
- moved D7 2.26 mm to (98.5, 93.3)
- moved D8 2.26 mm to (97.1, 74.5)
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Routing:
- net GND: track 272.9 -> 362.3 mm
- net Net-(J6-Pin_1): track 14.8 -> 77.0 mm
- net Net-(J6-Pin_2): track 22.6 -> 81.1 mm
- net +5V: track 283.0 -> 335.4 mm

Commit message: Add files via upload
Routing:
- net Net-(J6-Pin_1): track 77.0 -> 105.1 mm
- net Net-(J6-Pin_2): track 81.1 -> 82.2 mm, vias 0 -> 1
Changed lines of the file:
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@@
+	)
+	(segment
+		(start 196.55 65.78)
+		(end 199.65 62.68)
+		(width 2)
+		(layer "B.Cu")
+		(net "Net-(J6-Pin_1)")
 	)
 	(segment
@@
 		(start 199.73125 53.2175)
 		(end 195.4925 53.2175)
+		(width 2)
+		(layer "B.Cu")
+		(net "Net-(J6-Pin_1)")
+	)
+	(segment
+		(start 187.24 65.78)
+		(end 196.55 65.78)
 		(width 2)
 		(layer "B.Cu")
@@
 	)
 	(segment
+		(start 183.7425 62.2825)
+		(end 187.24 65.78)
+		(width 2)
+		(layer "B.Cu")
+		(net "Net-(J6-Pin_1)")
+	)
+	(segment
 		(start 195.4925 53.2175)
 		(end 195.4925 46.0325)
+		(width 2)
+		(layer "B.Cu")
+		(net "Net-(J6-Pin_1)")
+	)
+	(segment
+		(start 199.65 53.29875)
+		(end 199.73125 53.2175)
 		(width 2)
 		(layer "B.Cu")
@@
 	)
 	(segment
-		(start 187.28 101.58625)
-		(end 204.32 84.54625)
+		(start 199.65 62.68)
+		(end 199.65 53.29875)
+		(width 2)
+		(layer "B.Cu")
+		(net "Net-(J6-Pin_1)")
+	)
+	(segment
+		(start 190.4425 64.1325)
+		(end 192.07 65.76)
+		(width 2)
+		(layer "F.Cu")
+		(net "Net-(J6-Pin_2)")
+	)
+	(segment
+		(start 203.76 65.76)
+		(end 204.62 66.62)
+		(width 2)
+		(layer "F.Cu")
+		(net "Net-(J6-Pin_2)")
+	)
+	(segment
+		(start 190.4425 61.9075)
+		(end 190.4425 64.1325)
+		(width 2)
+		(layer "F.Cu")
+		(net "Net-(J6-Pin_2)")
+	)
+	(segment
+		(start 192.07 65.76)
+		(end 203.76 65.76)
+		(width 2)
+		(layer "F.Cu")
+		(net "Net-(J6-Pin_2)")
+	)
+	(via
+		(at 204.62 66.62)
+		(size 2)
+		(drill 1)
+		(layers "F.Cu" "B.Cu")
+		(net "Net-(J6-Pin_2)")
+	)
+	(segment
+		(start 204.62 84.24625)
+		(end 187.28 101.58625)
 		(width 2)
 		(layer "B.Cu")
@@
 	)
 	(segment
-		(start 200.74 65.07625)
-		(end 190.52 65.07625)
+		(start 204.62 66.62)
+		(end 204.62 84.24625)
 		(width 2)
 		(layer "B.Cu")
@@
 	)
 	(segment
-		(start 190.52 65.07625)
-		(end 190.4425 64.99875)
-		(width 2)
-		(layer "B.Cu")
-		(net "Net-(J6-Pin_2)")
-	)
-	(segment
-		(start 204.32 84.54625)
-		(end 204.32 68.65625)
-		(width 2)
-		(layer "B.Cu")
-		(net "Net-(J6-Pin_2)")
-	)
-	(segment
 		(start 183.7425 46.0325)
 		(end 190.4925 46.0325)
-		(width 2)
-		(layer "B.Cu")
-		(net "Net-(J6-Pin_2)")
-	)
-	(segment
-		(start 190.4425 64.99875)
-		(end 190.4425 61.9075)
 		(width 2)
 		(layer "B.Cu")
@@
 		(width 2)
 		(layer "B.Cu")
-		(net "Net-(J6-Pin_2)")
-	)
-	(segment
-		(start 204.32 68.65625)
-		(end 200.74 65.07625)
-		(width 2)
-		(layer "B.Cu")
