File: 4ch-relay-1fan-arduino-nano-pcb.kicad_pcb (KiCad board)
At the start: 2 copper layers, 62 parts, among them J1 Screw_Terminal_01x03, J2 Conn_01x08_Pin, J3 Screw_Terminal_01x03, J4 Screw_Terminal_01x03, J5 Screw_Terminal_01x03, J7 Conn_01x07_Pin, J9 Conn_01x04_Pin, K1 Relay_SPDT, K2 Relay_SPDT, K3 Relay_SPDT, K4 Relay_SPDT, Q1 2N3904, Q2 2N3904, Q3 2N3904, Q4 2N3904, Q5 BT136, U1 PC817, U2 PC817, U3 PC817, U4 PC817, U5 MOC3021M, U6 PC817, U7 TSOP1738, U8 HLK-10M05

Commit message: Add files via upload
Routing:
- net Net-(A1-D6): track 54.8 -> 55.5 mm
Changed lines of the file:
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@@
 	)
 	(segment
-		(start 123.7725 102.2025)
-		(end 123.7725 108.1525)
+		(start 108.5 99.3275)
+		(end 121.9975 99.3275)
+		(width 1)
+		(layer "B.Cu")
+		(net "Net-(A1-D6)")
+	)
+	(segment
+		(start 121.9975 99.3275)
+		(end 123.7725 101.1025)
 		(width 1)
 		(layer "B.Cu")
@@
 	)
 	(segment
-		(start 120.8975 99.3275)
-		(end 123.7725 102.2025)
+		(start 106.75 97.5775)
+		(end 108.5 99.3275)
 		(width 1)
 		(layer "B.Cu")
@@
 	)
 	(segment
-		(start 108.5 99.3275)
-		(end 120.8975 99.3275)
+		(start 123.7725 101.1025)
+		(end 123.7725 108.1525)
 		(width 1)
 		(layer "B.Cu")
@@
 		(layer "B.Cu")
 		(net "Net-(A1-D6)")
-	)
-	(segment
-		(start 106.75 97.5775)
-		(end 108.5 99.3275)
-		(width 1)
-		(layer "B.Cu")
-		(net "Net-(A1-D6)")

Commit message: Add files via upload
Parts:
- moved J7 1.25 mm to (151.4, 140.1)
- moved J9 1.25 mm to (111.5, 140.0)
- moved REF** 1.25 mm to (78.5, 145.9)
- moved D1 1.25 mm to (167.8, 92.1)
- moved D3 1.25 mm to (145.1, 91.8)
- moved D5 1.25 mm to (122.3, 92.1)
- moved J2 1.25 mm to (134.3, 107.0)
- moved R1 1.25 mm to (167.9, 87.3)
- moved R2 1.25 mm to (164.4, 82.5)
- moved R3 1.25 mm to (154.1, 88.6)
- moved R4 1.25 mm to (153.3, 95.8)
- moved R5 1.25 mm to (130.5, 95.8)
- moved R6 1.25 mm to (141.6, 82.5)
- moved R7 1.25 mm to (145.1, 87.1)
- moved R8 1.25 mm to (130.6, 88.6)
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Other:
- board outline added: 144.3 x 112.6 mm
- board text added: "CO"
- board text added: "Fan"
- board text added: "L"
- board text added: "N"
- board text added: "NC"

Commit message: Add files via upload
Other:
- board text added: "NO"
Changed lines of the file:
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@@
 		)
 	)
-	(gr_text "NC"
+	(gr_text "NO"
 		(at 97.805 40.235 90)
 		(layer "F.SilkS")
@@
 		)
 	)
-	(gr_text "NC"
+	(gr_text "NO"
 		(at 121.14 40.3125 90)
 		(layer "F.SilkS")
@@
 		)
 	)
-	(gr_text "NC"
+	(gr_text "NO"
 		(at 144.055 40.235 90)
 		(layer "F.SilkS")
@@
 		)
 	)
-	(gr_text "NC"
+	(gr_text "NO"
 		(at 167.465 40.235 90)
 		(layer "F.SilkS")

Commit message: Add files via upload
Other:
- board text added: "5v G R1 R2 R3 R4 ZC T"
- board text added: "5v G Tx Rx"
- board text added: "G S1 S2 S3 S4 DN UP"
Changed lines of the file:
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@@
 		(filling no)
 		(pcbplotparams
-			(layerselection 0x00000000_00000000_5555555d_5755f5ff)
+			(layerselection 0x00000000_00000000_5555555d_575555ff)
 			(plot_on_all_layers_selection 0x00000000_00000000_00000000_00000000)
 			(disableapertmacros no)
@@
 			(at 1.27 -3.96 0)
 			(layer "F.SilkS")
+			(hide yes)
 			(effects
 				(font
@@
 			(at 7.62 -5.08 90)
 			(layer "F.SilkS")
+			(hide yes)
 			(effects
 				(font
@@
 			(at 3.08 -2.47 0)
 			(layer "F.SilkS")
+			(hide yes)
 			(effects
 				(font
@@
 			(at 6 -4.2 0)
 			(layer "F.SilkS")
+			(hide yes)
 			(effects
 				(font
@@
 			(at 5.08 -2.37 90)
 			(layer "F.SilkS")
+			(hide yes)
 			(effects
 				(font
@@
 			(at 1.27 -3.96 0)
 			(layer "F.SilkS")
+			(hide yes)
 			(effects
 				(font
@@
 			(at 1.27 -3.56 90)
 			(layer "F.SilkS")
+			(hide yes)
 			(effects
 				(font
@@
 			(at 5.08 -2.37 0)
 			(layer "F.SilkS")
+			(hide yes)
 			(effects
 				(font
@@
 			(at 3.81 -2.33 90)
 			(layer "F.SilkS")
+			(hide yes)
 			(effects
 				(font
@@
 			(at 5.33 -2.25 90)
 			(layer "F.SilkS")
+			(hide yes)
 			(effects
 				(font
@@
 			(at 1.27 -2.37 90)
 			(layer "F.SilkS")
+			(hide yes)
 			(effects
 				(font
@@
 			(at 0 -2.38 90)
 			(layer "F.SilkS")
+			(hide yes)
 			(effects
 				(font
@@
 			(at 1.27 -3.56 90)
 			(layer "F.SilkS")
+			(hide yes)
 			(effects
 				(font
@@
 			(at 5.08 -2.37 0)
 			(layer "F.SilkS")
+			(hide yes)
 			(effects
 				(font
@@
 			(at 5.08 -2.47 0)
 			(layer "F.SilkS")
+			(hide yes)
 			(effects
 				(font
@@
 			(at 1.27 -2.37 90)
 			(layer "F.SilkS")
+			(hide yes)
 			(effects
 				(font
@@
 			(at 3.81 -2.33 90)
 			(layer "F.SilkS")
+			(hide yes)
 			(effects
 				(font
@@
 			(at 5.08 -2.37 90)
 			(layer "F.SilkS")
+			(hide yes)
 			(effects
 				(font
@@
 			(at 1.27 -3.56 90)
 			(layer "F.SilkS")
+			(hide yes)
 			(effects
 				(font
@@
 			(at 5.08 -2.37 90)
 			(layer "F.SilkS")
+			(hide yes)
 			(effects
 				(font
@@
 			(at 6 -4.2 0)
 			(layer "F.SilkS")
+			(hide yes)
 			(effects
 				(font
@@
 			(at 3.81 -2.33 90)
 			(layer "F.SilkS")
+			(hide yes)
 			(effects
 				(font
@@
 		)
 		(property "Value" "PC817"
-			(at -11.06 -1.52 90)
+			(at -2.165 1.465 180)
 			(layer "F.Fab")
 			(effects
@@
 			(at 3.81 -2.33 0)
 			(layer "F.SilkS")
+			(hide yes)
 			(effects
 				(font
@@
 			(at 21.25 -12.3 90)
 			(layer "F.SilkS")
+			(hide yes)
 			(effects
 				(font
@@
 			(at 5.08 -2.37 0)
 			(layer "F.SilkS")
+			(hide yes)
 			(effects
 				(font
@@
 			(at 5.08 -2.37 90)
 			(layer "F.SilkS")
+			(hide yes)
 			(effects
 				(font
@@
 			(at 5.08 -2.37 0)
 			(layer "F.SilkS")
+			(hide yes)
 			(effects
 				(font
@@
 			(at 1.27 -3.56 90)
 			(layer "F.SilkS")
+			(hide yes)
 			(effects
 				(font
@@
 			(at 2.54 -2.37 90)
 			(layer "F.SilkS")
+			(hide yes)
 			(effects
 				(font
@@
 			(at 5.08 -2.37 90)
 			(layer "F.SilkS")
+			(hide yes)
 			(effects
 				(font
@@
 			(at 2.54 -4.1 0)
 			(layer "F.SilkS")
+			(hide yes)
 			(effects
 				(font
@@
 			(at 5.08 -2.37 90)
 			(layer "F.SilkS")
+			(hide yes)
 			(effects
 				(font
@@
 			(at 6 -4.2 0)
 			(layer "F.SilkS")
+			(hide yes)
 			(effects
 				(font
@@
 			(at 1.27 -2.37 90)
 			(layer "F.SilkS")
+			(hide yes)
 			(effects
 				(font
@@
 			(at 5.08 -2.37 90)
 			(layer "F.SilkS")
+			(hide yes)
 			(effects
 				(font
@@
 			(at 3.81 -2.33 90)
 			(layer "F.SilkS")
+			(hide yes)
 			(effects
 				(font
@@
 			(at -0.645 -5.635 90)
 			(layer "F.SilkS")
+			(hide yes)
 			(effects
 				(font
@@
 			(at 5.08 -2.37 90)
 			(layer "F.SilkS")
+			(hide yes)
 			(effects
 				(font
@@
 			(at 5.08 -2.37 90)
 			(layer "F.SilkS")
+			(hide yes)
 			(effects
 				(font
@@
 			(at 3.81 -2.33 90)
 			(layer "F.SilkS")
+			(hide yes)
 			(effects
 				(font
@@
 			(at 2.54 -2.37 90)
 			(layer "F.SilkS")
+			(hide yes)
 			(effects
 				(font
@@
 			(at 1.27 -3.96 0)
 			(layer "F.SilkS")
+			(hide yes)
 			(effects
 				(font
@@
 			(at 1.27 -3.96 0)
 			(layer "F.SilkS")
+			(hide yes)
 			(effects
 				(font
@@
 			(at 5.08 -2.47 0)
 			(layer "F.SilkS")
+			(hide yes)
 			(effects
 				(font
@@
 			(at 5.08 -6.32 0)
 			(layer "F.SilkS")
+			(hide yes)
 			(effects
 				(font
@@
 			(at 5.08 -2.37 90)
 			(layer "F.SilkS")
+			(hide yes)
 			(effects
 				(font
@@
 			(at 5 -3.75 90)
 			(layer "F.SilkS")
+			(hide yes)
 			(effects
 				(font
@@
 			(at 6 -4.2 0)
 			(layer "F.SilkS")
+			(hide yes)
 			(effects
 				(font
@@
 			(at 5.08 -2.37 90)
 			(layer "F.SilkS")
+			(hide yes)
 			(effects
 				(font
@@
 			(at 5.08 -2.47 0)
 			(layer "F.SilkS")
+			(hide yes)
 			(effects
 				(font
@@
 		)
 	)
+	(gr_text "5v  G  Tx  Rx"
+		(at 110.14 143.55 0)
+		(layer "F.SilkS")
+		(effects
+			(font
+				(size 1 1)
+				(thickness 0.1)
+			)
+			(justify left bottom)
+		)
+	)
+	(gr_text "5v G R1 R2 R3 R4 ZC T"
+		(at 116.05 110.63 0)
+		(layer "F.SilkS")
+		(effects
+			(font
+				(size 1 1)
+				(thickness 0.1)
+			)
+			(justify left bottom)
+		)
+	)
+	(gr_text "G S1 S2 S3 S4 DN UP"
+		(at 135.63 144.02 0)
+		(layer "F.SilkS")
+		(effects
+			(font
+				(size 1 1)
+				(thickness 0.1)
+			)
+			(justify left bottom)
+		)
+	)
 	(gr_text "SASoftwareS"
 		(at 155.155 147.38875 0)
@@
 	(segment
 		(start 93.695 95.815)
-		(end 89.365 95.815)
-		(width 1)
-		(layer "B.Cu")
-		(net "Net-(R13-Pad2)")
-	)
-	(segment
-		(start 89.365 95.815)
-		(end 88.365 94.815)
+		(end 89.825 95.815)
 		(width 1)
 		(layer "B.Cu")
@@
 	)
 	(segment
-		(start 88.365 94.815)
+		(start 89.825 95.815)
 		(end 88.595 94.585)
 		(width 1)

Commit message: Add files via upload
Other:
- board text added: "Arduino_Nano_v3.x"
Changed lines of the file:
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@@
+		)
+	)
+	(gr_text "Arduino_Nano_v3.x"
+		(at 128.66 122.73 0)
+		(layer "F.SilkS")
+		(effects
+			(font
+				(size 1 1)
+				(thickness 0.1)
+			)
+			(justify left bottom)
 		)
 	)
